File: Hardware/KiCad/motor.kicad_sch (KiCad schematic)
At the start: 5 parts, among them U101 TB6612FNG

Commit message: change to pinout of atemega for PWM Motor 1
Parts:
- renumbered C106 to C_md1_1, C9 to C_md1_2, C108 to C_md1_3, C10 to C_md1_4, U101 to MOTOR_D_1
Changed lines of the file:
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@@
 (kicad_sch
-	(version 20231120)
+	(version 20250114)
 	(generator "eeschema")
-	(generator_version "8.0")
+	(generator_version "9.0")
 	(paper "A4")
 	(junction
@@
 	(label "a_2"
 		(at 73.66 45.72 0)
-		(fields_autoplaced yes)
 		(effects
 			(font
@@
 	(label "pwm_1"
 		(at 73.66 48.26 0)
-		(fields_autoplaced yes)
 		(effects
 			(font
@@
 	(label "b_1"
 		(at 73.66 52.07 0)
-		(fields_autoplaced yes)
 		(effects
 			(font
@@
 	(label "vcc"
 		(at 114.3 40.64 0)
-		(fields_autoplaced yes)
 		(effects
 			(font
@@
 	(label "vm"
 		(at 114.3 48.26 0)
-		(fields_autoplaced yes)
 		(effects
 			(font
@@
 	(label "b_2"
 		(at 73.66 54.61 0)
-		(fields_autoplaced yes)
 		(effects
 			(font
@@
 	(label "pwm_1"
 		(at 73.66 57.15 0)
-		(fields_autoplaced yes)
 		(effects
 			(font
@@
 	(label "ao_2"
 		(at 114.3 60.96 0)
-		(fields_autoplaced yes)
 		(effects
 			(font
@@
 	(label "a_1"
 		(at 73.66 43.18 0)
-		(fields_autoplaced yes)
 		(effects
 			(font
@@
 	(label "bo_2"
 		(at 114.3 74.93 0)
-		(fields_autoplaced yes)
 		(effects
 			(font
@@
 	(label "bo_1"
 		(at 114.3 68.58 0)
-		(fields_autoplaced yes)
 		(effects
 			(font
@@
 	(label "ao_1"
 		(at 114.3 54.61 0)
-		(fields_autoplaced yes)
 		(effects
 			(font
@@
 		(shape output)
 		(at 137.16 60.96 0)
-		(fields_autoplaced yes)
 		(effects
 			(font
@@
 		(shape input)
 		(at 137.16 71.12 0)
-		(fields_autoplaced yes)
 		(effects
 			(font
@@
 		(shape input)
 		(at 48.26 50.8 180)
-		(fields_autoplaced yes)
 		(effects
 			(font
@@
 		(shape input)
 		(at 41.91 46.99 180)
-		(fields_autoplaced yes)
 		(effects
 			(font
@@
 		(shape input)
 		(at 58.42 57.15 180)
-		(fields_autoplaced yes)
 		(effects
 			(font
@@
 		(dnp no)
 		(fields_autoplaced yes)
-		(property "Reference" "C106"
+		(property "Reference" "C_md1_1"
 			(at 156.21 39.3762 0)
 			(effects
@@
 		(dnp no)
 		(fields_autoplaced yes)
-		(property "Reference" "C10"
+		(property "Reference" "C_md1_4"
 			(at 171.45 70.5738 0)
 			(effects
@@
 		(dnp no)
 		(fields_autoplaced yes)
-		(property "Reference" "#PWR0107"
+		(property "Reference" "#PWR09"
 			(at 73.66 60.96 0)
 			(effects
@@
 		(dnp no)
 		(fields_autoplaced yes)
-		(property "Reference" "#PWR0128"
+		(property "Reference" "#PWR012"
 			(at 153.67 54.61 0)
 			(effects
@@
 		(dnp no)
 		(fields_autoplaced yes)
-		(property "Reference" "U101"
+		(property "Reference" "MOTOR_D_1"
 			(at 96.52 33.02 0)
 			(effects
@@
 		(dnp no)
 		(fields_autoplaced yes)
-		(property "Reference" "#PWR0106"
+		(property "Reference" "#PWR014"
 			(at 153.67 86.36 0)
 			(effects
@@
 		(dnp no)
 		(fields_autoplaced yes)
-		(property "Reference" "C9"
+		(property "Reference" "C_md1_2"
 			(at 156.21 71.1262 0)
 			(effects
@@
 		(dnp no)
 		(fields_autoplaced yes)
-		(property "Reference" "#PWR0129"
+		(property "Reference" "#PWR013"
 			(at 153.67 68.58 0)
 			(effects
@@
 		(dnp no)
 		(fields_autoplaced yes)
-		(property "Reference" "#PWR0127"
+		(property "Reference" "#PWR011"
 			(at 153.67 36.83 0)
 			(effects
@@
 		(dnp no)
 		(fields_autoplaced yes)
-		(property "Reference" "#PWR0108"
+		(property "Reference" "#PWR010"
 			(at 81.28 90.17 0)
 			(effects
@@
 		(dnp no)
 		(fields_autoplaced yes)
-		(property "Reference" "C108"
+		(property "Reference" "C_md1_3"
 			(at 171.45 38.8238 0)
 			(effects
