File: Hardware/KiCad/starter.kicad_sch (KiCad schematic)
At the start: 1 part

Commit message: change to pinout of atemega for PWM Motor 1
Changed lines of the file:
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@@
 (kicad_sch
-	(version 20231120)
+	(version 20250114)
 	(generator "eeschema")
-	(generator_version "8.0")
+	(generator_version "9.0")
 	(paper "A4")
 	(wire
@@
 		(shape input)
 		(at 81.28 74.93 180)
-		(fields_autoplaced yes)
 		(effects
 			(font
