File: Hardware/KiCad/voltage_regulator_sch.kicad_sch (KiCad schematic)
At the start: 5 parts, among them U100 LM1117DT-5.0

Commit message: change to pinout of atemega for PWM Motor 1
Parts:
- renumbered C11 to C1, C12 to C2, U100 to VOLTAGE_STAB1
Changed lines of the file:
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@@
 (kicad_sch
-	(version 20231120)
+	(version 20250114)
 	(generator "eeschema")
-	(generator_version "8.0")
+	(generator_version "9.0")
 	(paper "A4")
 	(junction
@@
 	(label "GND"
 		(at 118.11 46.99 0)
-		(fields_autoplaced yes)
 		(effects
 			(font
@@
 	(label "S_PMOS"
 		(at 95.25 38.1 0)
-		(fields_autoplaced yes)
 		(effects
 			(font
@@
 	(label "GND"
 		(at 72.39 53.34 0)
-		(fields_autoplaced yes)
 		(effects
 			(font
@@
 	(label "VI"
 		(at 107.95 38.1 0)
-		(fields_autoplaced yes)
 		(effects
 			(font
@@
 	(label "V0"
 		(at 127 38.1 0)
-		(fields_autoplaced yes)
 		(effects
 			(font
@@
 	(label "GND"
 		(at 88.9 53.34 0)
-		(fields_autoplaced yes)
 		(effects
 			(font
@@
 	(label "D_PMOS"
 		(at 74.93 38.1 0)
-		(fields_autoplaced yes)
 		(effects
 			(font
@@
 		(dnp no)
 		(fields_autoplaced yes)
-		(property "Reference" "#PWR0119"
+		(property "Reference" "#PWR024"
 			(at 118.11 54.61 0)
 			(effects
@@
 		(on_board yes)
 		(dnp no)
-		(property "Reference" "C11"
+		(property "Reference" "C1"
 			(at 107.188 42.672 0)
 			(effects
@@
 		(dnp no)
 		(fields_autoplaced yes)
-		(property "Reference" "#PWR0100"
+		(property "Reference" "#PWR025"
 			(at 129.54 39.37 0)
 			(effects
@@
 		(dnp no)
 		(fields_autoplaced yes)
-		(property "Reference" "#PWR0101"
+		(property "Reference" "#PWR026"
 			(at 129.54 53.34 0)
 			(effects
@@
 		(on_board yes)
 		(dnp no)
-		(property "Reference" "C12"
+		(property "Reference" "C2"
 			(at 130.81 42.418 0)
 			(effects
@@
 		(dnp no)
 		(fields_autoplaced yes)
-		(property "Reference" "#PWR0112"
+		(property "Reference" "#PWR023"
 			(at 106.68 53.34 0)
 			(effects
@@
 		(dnp no)
 		(fields_autoplaced yes)
-		(property "Reference" "#PWR0111"
+		(property "Reference" "#PWR022"
 			(at 106.68 39.37 0)
 			(effects
@@
 		(dnp no)
 		(fields_autoplaced yes)
-		(property "Reference" "U100"
+		(property "Reference" "VOLTAGE_STAB1"
 			(at 118.11 31.75 0)
 			(effects
